File: hardware/BFS9000 switch plate/BFS9000 switch plate.kicad_pcb (KiCad board)
At the start: 2 copper layers, 252.4 x 149.4 mm, 88 parts

Commit message: fix(BFS9000 switch plate): update date and position of text component
Parts:
- added BFS9000_Back: LOGO, BFS9000:BFS9000+Gran Canaria, B.Cu at (219.9, 84.0)
- added BFS9000_Front: LOGO, BFS9000:BFS9000+Gran Canaria, F.Cu at (222.4, 84.3)
Routing:
- removed copper zone on B.Cu, net GND
- removed copper zone on F.Cu, net VSYS
Other:
- outline, holes or cut-outs redrawn
- board text added: "2024/04/10 23:12"
- board text added: "Dedicado a mi hijo Marco"
