File: hardware/BFS9000 bottom plate/BFS9000 bottom plate.kicad_pcb (KiCad board)
At the start: 2 copper layers, 252.5 x 149.4 mm, 29 parts

Commit message: fix(BFS9000 switch plate): update plot output directory and layer selection in PCB files
Routing:
- removed copper zone on B.Cu, net GND
- removed copper zone on F.Cu, net VSYS
Changed lines of the file:
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@@
 		(grid_origin 139.93 122.442)
 		(pcbplotparams
-			(layerselection 0x00000000_00000000_55555555_57555550)
+			(layerselection 0x00000000_00000000_55555555_5755f5ff)
 			(plot_on_all_layers_selection 0x00000000_00000000_00000000_00000008)
 			(disableapertmacros no)
@@
 			(plotpadnumbers no)
 			(hidednponfab no)
-			(sketchdnponfab no)
-			(crossoutdnponfab no)
+			(sketchdnponfab yes)
+			(crossoutdnponfab yes)
 			(subtractmaskfromsilk no)
-			(outputformat 3)
+			(outputformat 1)
 			(mirror no)
 			(drillshape 0)
@@
 		(layer "Edge.Cuts")
 	)
-	(zone
-		(net "VSYS")
-		(layer "F.Cu")
-		(hatch edge 0.5)
-		(priority 1)
-		(connect_pads yes
-			(clearance 0.3)
-		)
-		(min_thickness 0.25)
-		(fill yes
-			(thermal_gap 0.5)
-			(thermal_bridge_width 0.5)
-			(island_removal_mode 0)
-		)
-		(polygon
-			(pts
-				(xy 60.58 35.24955) (xy 283.47755 35.24955) (xy 322.26 74.032) (xy 322.26 142.322) (xy 294.84 169.742)
-				(xy 294.84 206.882) (xy 233.14 206.882) (xy 225.99 199.732) (xy 63.15 199.732) (xy 51.01245 187.59445)
-				(xy 51.01245 44.8171)
-			)
-		)
-	)
-	(zone
-		(net "GND")
-		(layer "B.Cu")
-		(hatch edge 0.5)
-		(priority 1)
-		(connect_pads yes
-			(clearance 0.25)
-		)
-		(min_thickness 0.25)
-		(fill yes
-			(thermal_gap 0.5)
-			(thermal_bridge_width 0.5)
-			(island_removal_mode 0)
-		)
-		(polygon
-			(pts
-				(xy 60.58 35.24955) (xy 283.47755 35.24955) (xy 322.26 74.032) (xy 322.26 142.322) (xy 294.84 169.742)
-				(xy 294.84 206.882) (xy 233.14 206.882) (xy 225.99 199.732) (xy 63.15 199.732) (xy 51.01245 187.59445)
-				(xy 51.01245 44.8171)
-			)
-		)
-	)
 	(embedded_fonts no)
