File: hardware/BFS9000/BFS9000.kicad_pcb (KiCad board)
At the start: 2 copper layers, 252.5 x 149.4 mm, 38 parts

Commit message: feat(hardware): add footprints for all switches
Parts:
- added C0R0: MX_SW_HS, BFS9000:Cherry_MX_DS_Hotswap_Vertical, B.Cu at (301.3, 97.2)
- added C0R1: MX_SW_HS, BFS9000:Cherry_MX_DS_Hotswap_Vertical, B.Cu at (293.9, 124.8)
- added C0R3: MX_SW_HS, BFS9000:Cherry_MX_DS_Hotswap_Vertical, B.Cu at (284.0, 161.5)
- added C0R5: MX_SW_HS, BFS9000:Cherry_MX_DS_Hotswap_Vertical, B.Cu at (276.6, 189.1)
- added C10R5: MX_SW_HS, BFS9000:Cherry_MX_DS_Hotswap_Vertical, B.Cu at (77.9, 178.3)
- added C1R0: MX_SW_HS, BFS9000:Cherry_MX_DS_Hotswap_Vertical, B.Cu at (284.0, 88.0)
- added C1R1: MX_SW_HS, BFS9000:Cherry_MX_DS_Hotswap_Vertical, B.Cu at (279.1, 106.4)
- added C1R2: MX_SW_HS, BFS9000:Cherry_MX_DS_Hotswap_Vertical, B.Cu at (274.1, 124.8)
- added C1R3: MX_SW_HS, BFS9000:Cherry_MX_DS_Hotswap_Vertical, B.Cu at (269.2, 143.2)
- added C1R4: MX_SW_HS, BFS9000:Cherry_MX_DS_Hotswap_Vertical, B.Cu at (264.3, 161.6)
- added C1R5: MX_SW_HS, BFS9000:Cherry_MX_DS_Hotswap_Vertical, B.Cu at (259.3, 180.0)
- added C2R0: MX_SW_HS, BFS9000:Cherry_MX_DS_Hotswap_Vertical, B.Cu at (266.2, 80.7)
- added C2R1: MX_SW_HS, BFS9000:Cherry_MX_DS_Hotswap_Vertical, B.Cu at (261.3, 99.1)
- added C2R2: MX_SW_HS, BFS9000:Cherry_MX_DS_Hotswap_Vertical, B.Cu at (256.4, 117.5)
- added C2R3: MX_SW_HS, BFS9000:Cherry_MX_DS_Hotswap_Vertical, B.Cu at (251.5, 135.9)
- added C2R4: MX_SW_HS, BFS9000:Cherry_MX_DS_Hotswap_Vertical, B.Cu at (246.5, 154.3)
- added C2R5: MX_SW_HS, BFS9000:Cherry_MX_DS_Hotswap_Vertical, B.Cu at (241.6, 172.7)
- added C3R0: MX_SW_HS, BFS9000:Cherry_MX_DS_Hotswap_Vertical, B.Cu at (247.2, 78.1)
- added C3R1: MX_SW_HS, BFS9000:Cherry_MX_DS_Hotswap_Vertical, B.Cu at (242.3, 96.5)
- added C3R2: MX_SW_HS, BFS9000:Cherry_MX_DS_Hotswap_Vertical, B.Cu at (237.3, 114.9)
- added C3R3: MX_SW_HS, BFS9000:Cherry_MX_DS_Hotswap_Vertical, B.Cu at (232.4, 133.3)
- added C3R4: MX_SW_HS, BFS9000:Cherry_MX_DS_Hotswap_Vertical, B.Cu at (227.5, 151.7)
- added C3R5: MX_SW_HS, BFS9000:Cherry_MX_DS_Hotswap_Vertical, B.Cu at (222.5, 170.1)
- added C4R0: MX_SW_HS, BFS9000:Cherry_MX_DS_Hotswap_Vertical, B.Cu at (197.1, 72.2)
- added C4R1: MX_SW_HS, BFS9000:Cherry_MX_DS_Hotswap_Vertical, B.Cu at (197.1, 91.2)
- added C4R2: MX_SW_HS, BFS9000:Cherry_MX_DS_Hotswap_Vertical, B.Cu at (197.1, 110.2)
- added C4R3: MX_SW_HS, BFS9000:Cherry_MX_DS_Hotswap_Vertical, B.Cu at (197.1, 129.3)
- added C4R4: MX_SW_HS, BFS9000:Cherry_MX_DS_Hotswap_Vertical, B.Cu at (197.1, 148.3)
- added C5R0: MX_SW_HS, BFS9000:Cherry_MX_DS_Hotswap_Vertical, B.Cu at (178.0, 72.2)
- added C5R03: MX_SW_HS, BFS9000:Cherry_MX_DS_Hotswap_Vertical, B.Cu at (178.0, 129.3)
- added C5R1: MX_SW_HS, BFS9000:Cherry_MX_DS_Hotswap_Vertical, B.Cu at (178.0, 91.2)
- added C5R2: MX_SW_HS, BFS9000:Cherry_MX_DS_Hotswap_Vertical, B.Cu at (178.0, 110.2)
- added C5R4: MX_SW_HS, BFS9000:Cherry_MX_DS_Hotswap_Vertical, B.Cu at (178.0, 148.3)
- added C6R0: MX_SW_HS, BFS9000:Cherry_MX_DS_Hotswap_Vertical, B.Cu at (159.0, 67.8)
- added C6R1: MX_SW_HS, BFS9000:Cherry_MX_DS_Hotswap_Vertical, B.Cu at (159.0, 86.8)
- added C6R2: MX_SW_HS, BFS9000:Cherry_MX_DS_Hotswap_Vertical, B.Cu at (159.0, 105.9)
- added C6R3: MX_SW_HS, BFS9000:Cherry_MX_DS_Hotswap_Vertical, B.Cu at (159.0, 124.9)
- added C6R4: MX_SW_HS, BFS9000:Cherry_MX_DS_Hotswap_Vertical, B.Cu at (159.0, 144.0)
- added C6R5: MX_SW_HS, BFS9000:Cherry_MX_DS_Hotswap_Vertical, B.Cu at (159.0, 163.0)
- added C7R0: MX_SW_HS, BFS9000:Cherry_MX_DS_Hotswap_Vertical, B.Cu at (139.9, 65.3)
- added C7R1: MX_SW_HS, BFS9000:Cherry_MX_DS_Hotswap_Vertical, B.Cu at (139.9, 84.3)
- added C7R2: MX_SW_HS, BFS9000:Cherry_MX_DS_Hotswap_Vertical, B.Cu at (139.9, 103.4)
- added C7R3: MX_SW_HS, BFS9000:Cherry_MX_DS_Hotswap_Vertical, B.Cu at (139.9, 122.4)
- added C7R4: MX_SW_HS, BFS9000:Cherry_MX_DS_Hotswap_Vertical, B.Cu at (139.9, 141.5)
- added C7R5: MX_SW_HS, BFS9000:Cherry_MX_DS_Hotswap_Vertical, B.Cu at (139.9, 160.5)
- added C8R0: MX_SW_HS, BFS9000:Cherry_MX_DS_Hotswap_Vertical, B.Cu at (120.9, 67.8)
- added C8R1: MX_SW_HS, BFS9000:Cherry_MX_DS_Hotswap_Vertical, B.Cu at (120.9, 86.8)
- added C8R2: MX_SW_HS, BFS9000:Cherry_MX_DS_Hotswap_Vertical, B.Cu at (120.9, 105.9)
- added C8R3: MX_SW_HS, BFS9000:Cherry_MX_DS_Hotswap_Vertical, B.Cu at (120.9, 124.9)
- added C8R4: MX_SW_HS, BFS9000:Cherry_MX_DS_Hotswap_Vertical, B.Cu at (120.9, 144.0)
- added C8R5: MX_SW_HS, BFS9000:Cherry_MX_DS_Hotswap_Vertical, B.Cu at (120.9, 163.0)
- added C9R0: MX_SW_HS, BFS9000:Cherry_MX_DS_Hotswap_Vertical, B.Cu at (101.8, 69.7)
- added C9R1: MX_SW_HS, BFS9000:Cherry_MX_DS_Hotswap_Vertical, B.Cu at (101.8, 88.7)
- added C9R2: MX_SW_HS, BFS9000:Cherry_MX_DS_Hotswap_Vertical, B.Cu at (101.8, 107.8)
- added C9R3: MX_SW_HS, BFS9000:Cherry_MX_DS_Hotswap_Vertical, B.Cu at (101.8, 126.8)
- added C9R4: MX_SW_HS, BFS9000:Cherry_MX_DS_Hotswap_Vertical, B.Cu at (101.8, 145.9)
- added C9R5: MX_SW_HS, BFS9000:Cherry_MX_DS_Hotswap_Vertical, B.Cu at (98.2, 168.5)
- added ENC1: Rotary_Encoder_Switch-Device, BFS9000:RotaryEncoder_Alps_EC11E-Switch_Vertical_H20mm-keebio_modified, F.Cu at (81.6, 150.5)

Commit message: feat(hardware): add RP2040 footprint and peripheral circuitry
Add the RP2040 footprint, decoupling capacitors, OLED connectors, I2C pull-up resistors, and left/right keyboard side detection circuitry.
Parts:
- removed ENC1: Rotary_Encoder_Switch-Device, BFS9000:RotaryEncoder_Alps_EC11E-Switch_Vertical_H20mm-keebio_modified
- added C1: 1uF, Capacitor_SMD:C_0805_2012Metric_Pad1.18x1.45mm_HandSolder, F.Cu at (81.6, 86.9)
- added C2: 0.1uF, Capacitor_SMD:C_0805_2012Metric_Pad1.18x1.45mm_HandSolder, B.Cu at (71.8, 87.0)
- added C3: 0.1uF, Capacitor_SMD:C_0805_2012Metric_Pad1.18x1.45mm_HandSolder, B.Cu at (83.3, 141.1)
- added C4: 0.1uF, Capacitor_SMD:C_0805_2012Metric_Pad1.18x1.45mm_HandSolder, F.Cu at (79.2, 134.6)
- added D31: MBR120VLSF, Sofle_Pico:D_SOD-123_DO-41_7.62mm_Hybrid_DoubleSided, F.Cu at (63.4, 87.2)
- added D31_B: D_SOD-128, Diode_SMD:D_SOD-128, F.Cu at (63.4, 87.2)
- added J1: Conn_01x04, BFS9000:OLED SSD1306 128x64, F.Cu at (76.8, 102.4)
- added J3: Conn_01x04, BFS9000:Cirque tie in, B.Cu at (89.6, 127.9)
- added J6: Conn_01x01, Connector_PinHeader_2.54mm:PinHeader_1x01_P2.54mm_Vertical, B.Cu at (222.5, 81.5)
- added JP1: SolderJumper_2_Open, BFS9000:Level Shifter Bypass Jumper, B.Cu at (78.9, 137.1)
- added LEFT HAND: 2.2k, BFS9000:Res_1206_SMD_6.3mm_TH_Hybrid, B.Cu at (75.4, 166.2)
- added R3: 2.2k, BFS9000:Res_1206_SMD_6.3mm_TH_Hybrid, B.Cu at (75.0, 93.7)
- added R4: 2.2k, BFS9000:Res_1206_SMD_6.3mm_TH_Hybrid, B.Cu at (79.7, 93.8)
- added RIGHT HAND: 2.2k, BFS9000:Res_1206_SMD_6.3mm_TH_Hybrid, B.Cu at (75.3, 162.1)
- added U1: RP2040 Core board, BFS9000:RPi_Pico_SMD_TH_DS, F.Cu at (76.8, 107.5)
