File: hardware/BFS9000/BFS9000.kicad_pcb (KiCad board)
At the start: 2 copper layers, 252.5 x 149.4 mm, 237 parts, among them J1 Conn_01x04, J2 MJ-4PP-9, J3 Conn_01x04, J4 Conn_01x04, J5 Conn_01x01, J6 Conn_01x01, Q1 Si2301CDS, U1 RP2040 Core board

Commit message: feat(hardware): update BFS9000 schematic and PCB layout
Parts:
- BFS9000_Back, BFS9000_Front: footprint BFS9000:BFS9000+Gran Canaria -> BFS9000:Logo_BFS9000_Gran_Canaria
- C0R0, C0R1, C0R3, C0R5, C10R5, C1R0, C1R1, C1R2, C1R3, C1R4, C1R5, C2R0, C2R1, C2R2, C2R3, C2R4, C2R5, C3R0, C3R1, C3R2, C3R3, C3R4, C3R5, C4R0, C4R1, C4R2, C4R3, C4R4, C5R0, C5R1, C5R2, C5R4, C6R0, C6R1, C6R2, C6R3, C6R4, C6R5, C7R0, C7R1, C7R2, C7R3, C7R4, C7R5, C8R0, C8R1, C8R2, C8R3, C8R4, C8R5, C9R0, C9R1, C9R2, C9R3, C9R4, C9R5: footprint BFS9000:Cherry_MX_DS_Hotswap_Vertical -> BFS9000:SW_Cherry_MX_Hotswap_DS
- C1, C2, C3, C4: footprint Capacitor_SMD:C_0805_2012Metric_Pad1.18x1.45mm_HandSolder -> BFS9000:C_0805_HandSolder
- C5R3: renamed from C5R03; footprint BFS9000:Cherry_MX_DS_Hotswap_Vertical -> BFS9000:SW_Cherry_MX_Hotswap_DS
- Cut_1, Cut_10, Cut_11, Cut_12, Cut_13, Cut_14, Cut_2, Cut_3, Cut_4, Cut_5, Cut_6, Cut_7, Cut_8, Cut_9: footprint BFS9000:LongOvalCut -> BFS9000:Cutout_Long_Oval
- D31: footprint Sofle_Pico:D_SOD-123_DO-41_7.62mm_Hybrid_DoubleSided -> BFS9000:D_Hybrid_SOD-123_DO-41_P7.62mm_DS
- D31_B: footprint Diode_SMD:D_SOD-128 -> BFS9000:D_SOD-128
- DC0R0, DC0R1, DC0R3, DC0R5, DC10R5, DC1R0, DC1R1, DC1R2, DC1R3, DC1R4, DC1R5, DC2R0, DC2R1, DC2R2, DC2R3, DC2R4, DC2R5, DC3R0, DC3R1, DC3R2, DC3R3, DC3R4, DC3R5, DC4R0, DC4R1, DC4R2, DC4R3, DC4R4, DC5R0, DC5R1, DC5R2, DC5R4, DC6R0, DC6R1, DC6R2, DC6R3, DC6R4, DC6R5, DC7R0, DC7R1, DC7R2, DC7R3, DC7R4, DC7R5, DC8R0, DC8R1, DC8R2, DC8R3, DC8R4, DC8R5, DC9R0, DC9R1, DC9R2, DC9R3, DC9R4, DC9R5, rD1: footprint BFS9000:D_SOD-123_DO-35_Hybrid_DoubleSided_V2 -> BFS9000:D_Hybrid_SOD-123_DO-35_DS
- DC5R3: renamed from DC5R03; footprint BFS9000:D_SOD-123_DO-35_Hybrid_DoubleSided_V2 -> BFS9000:D_Hybrid_SOD-123_DO-35_DS
- ENC1: value Rotary_Encoder_Switch-Device -> Encoder_Rotary_Switch; footprint BFS9000:RotaryEncoder_Alps_EC11E-Switch_Vertical_H20mm-keebio_modified -> BFS9000:Encoder_EC11E_Switch_Vertical_H20mm
- J1: footprint BFS9000:OLED SSD1306 128x64 -> BFS9000:Display_OLED_SSD1306_128x64
- J3, J4: footprint BFS9000:Cirque tie in -> BFS9000:Conn_Touchpad
- J5, J6: footprint Connector_PinHeader_2.54mm:PinHeader_1x01_P2.54mm_Vertical -> BFS9000:PinHeader_1x01_P2.54mm
- JP1: footprint BFS9000:Level Shifter Bypass Jumper -> BFS9000:SolderJumper_Level_Shifter_Bypass
- LEFT_HAND1, R3, R4, RIGHT_HAND1: footprint BFS9000:Res_1206_SMD_6.3mm_TH_Hybrid -> BFS9000:R_Hybrid_1206_P6.3mm
- S1, S2: value MX_stab -> Stabilizer_MX; footprint PCM_marbastlib-mx:STAB_MX_2u -> BFS9000:Stabilizer_MX_2u
- TH1, TH2, TH4, TH5: footprint BFS9000:Hole from sofle for M2 posts gold rimmer narrow-keyplate-hole -> BFS9000:Mount_M2_Post_Hole_Keyplate_Narrow
- TH10, TH11, TH12, TH13, TH14, TH15, TH16, TH17, TH19, TH20, TH3, TH6, TH7, TH9: footprint BFS9000:Hole from sofle for M2 posts gold rimmer wide-keyplate-hole -> BFS9000:Mount_M2_Post_Hole_Keyplate_Wide
- TH18, TH8: footprint BFS9000:Tenting_Puck.kicad_mod_nocenter_v2 -> BFS9000:Mount_Tenting_Puck
- Wiki_Back, Wiki_Front: footprint BFS9000:Wiki-QR -> BFS9000:QR_Wiki
Routing:
- net row0: track 0.00 -> 488.0 mm, vias 0 -> 14
- net VSYS: track 0.00 -> 417.9 mm, vias 0 -> 171
- net col0: track 0.00 -> 380.3 mm, vias 0 -> 12
- net col2: track 0.00 -> 363.0 mm, vias 0 -> 18
- net col1: track 0.00 -> 354.6 mm, vias 0 -> 11
- net row5: track 0.00 -> 348.1 mm, vias 0 -> 3
- net col3: track 0.00 -> 304.9 mm, vias 0 -> 10
- net row3: track 0.00 -> 280.8 mm, vias 0 -> 1
- net row1: track 0.00 -> 272.5 mm, vias 0 -> 5
- net row4: track 0.00 -> 271.4 mm, vias 0 -> 1
- net LED_T: track 0.00 -> 263.4 mm, vias 0 -> 2
- net col4: track 0.00 -> 255.9 mm, vias 0 -> 6
- net col6: track 0.00 -> 241.9 mm, vias 0 -> 13
- net row2: track 0.00 -> 218.9 mm, vias 0 -> 4
- net col5: track 0.00 -> 207.1 mm, vias 0 -> 7
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Other:
- board text added: "Rev: 0.4"
- board text removed: "Rev: 0.3"
