File: hardware/BFS9000/Addressable RGB LEDs.kicad_sch (KiCad schematic)
At the start: 64 parts, among them J5 Conn_01x01, J6 Conn_01x01

Commit message: feat(hardware): update BFS9000 schematic and PCB layout
Parts:
- J5, J6: footprint Connector_PinHeader_2.54mm:PinHeader_1x01_P2.54mm_Vertical -> BFS9000:PinHeader_1x01_P2.54mm; symbol Connector_Generic:Conn_01x01 -> BFS9000:Conn_01x01
- MLED1, MLED10, MLED11, MLED12, MLED13, MLED14, MLED15, MLED16, MLED17, MLED18, MLED19, MLED2, MLED20, MLED21, MLED22, MLED23, MLED24, MLED25, MLED26, MLED27, MLED28, MLED29, MLED3, MLED4, MLED5, MLED6, MLED7, MLED8, MLED9, SLED1, SLED10, SLED11, SLED12, SLED13, SLED14, SLED15, SLED16, SLED17, SLED18, SLED19, SLED2, SLED20, SLED21, SLED22, SLED3, SLED4, SLED5, SLED6, SLED7, SLED8, SLED9, TLED1, TLED2, TLED3, TLED4, TLED5, TLED6: footprint BFS9000:Cust_SK6803_MINI-E_v3.5.5 -> BFS9000:Cust_SK6803_MINI-E_BFS9000; symbol Temp:SK6803MINIE_V2_COMPAT_N -> BFS9000:LED_SK6803MINI_E
- MULED1, MULED2, MULED3, SULED1, SULED2: footprint BFS9000:Cust_SK6803_MINI-E_v3.5.5 -> BFS9000:Cust_SK6803_MINI-E_BFS9000_Underglow; symbol Temp:SK6803MINIE_V2_COMPAT_N -> BFS9000:LED_SK6803MINI_E
